File: kicad/blackbox.kicad_sch (KiCad schematic)
At the start: 3 parts

Commit message: journal
Parts:
- renumbered C43 to C16, R39 to R13
Changed lines of the file:
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@@
 		(dnp no)
 		(fields_autoplaced yes)
-		(property "Reference" "#PWR0153"
+		(property "Reference" "#PWR040"
 			(at 95.25 49.53 0)
 			(hide yes)
@@
 			(project "Dreamscape-F405-2020"
 				(path "/97210a04-f116-4730-b66b-a4a0966edab8/505a8c64-a928-427e-9c04-823b276ca53f"
-					(reference "#PWR0153")
+					(reference "#PWR040")
 					(unit 1)
 				)
@@
 		(dnp no)
 		(fields_autoplaced yes)
-		(property "Reference" "#PWR0155"
+		(property "Reference" "#PWR038"
 			(at 74.93 43.18 0)
 			(hide yes)
@@
 			(project "Dreamscape-F405-2020"
 				(path "/97210a04-f116-4730-b66b-a4a0966edab8/505a8c64-a928-427e-9c04-823b276ca53f"
-					(reference "#PWR0155")
+					(reference "#PWR038")
 					(unit 1)
 				)
@@
 		(dnp no)
 		(fields_autoplaced yes)
-		(property "Reference" "#PWR0154"
+		(property "Reference" "#PWR039"
 			(at 74.93 73.66 0)
 			(hide yes)
@@
 			(project "Dreamscape-F405-2020"
 				(path "/97210a04-f116-4730-b66b-a4a0966edab8/505a8c64-a928-427e-9c04-823b276ca53f"
-					(reference "#PWR0154")
+					(reference "#PWR039")
 					(unit 1)
 				)
@@
 		(in_pos_files yes)
 		(dnp no)
-		(property "Reference" "C43"
+		(property "Reference" "C16"
 			(at 61.976 35.56 90)
 			(show_name no)
@@
 			(project "Dreamscape-F405-2020"
 				(path "/97210a04-f116-4730-b66b-a4a0966edab8/505a8c64-a928-427e-9c04-823b276ca53f"
-					(reference "C43")
+					(reference "C16")
 					(unit 1)
 				)
@@
 		(dnp no)
 		(fields_autoplaced yes)
-		(property "Reference" "#PWR060"
+		(property "Reference" "#PWR037"
 			(at 54.61 39.37 0)
 			(hide yes)
@@
 			(project "Dreamscape-F405-2020"
 				(path "/97210a04-f116-4730-b66b-a4a0966edab8/505a8c64-a928-427e-9c04-823b276ca53f"
-					(reference "#PWR060")
+					(reference "#PWR037")
 					(unit 1)
 				)
@@
 		(in_pos_files yes)
 		(dnp no)
-		(property "Reference" "R39"
+		(property "Reference" "R13"
 			(at 100.33 49.53 90)
 			(show_name no)
@@
 			(project "Dreamscape-F405-2020"
 				(path "/97210a04-f116-4730-b66b-a4a0966edab8/505a8c64-a928-427e-9c04-823b276ca53f"
-					(reference "R39")
+					(reference "R13")
 					(unit 1)
 				)
