File: kicad/pads.kicad_sch (KiCad schematic)
At the start: 46 parts, among them J1 5V, J10 5V, J11 5V, J12 5V, J13 5V, J14 5V, J15 5V, J16 5V, J17 5V, J18 5V, J19 5V, J2 5V, J20 5V, J21 5V, J22 5V, J23 5V, J24 5V, J25 5V, J26 5V, J27 5V, J28 5V, J29 5V, J3 5V, J30 5V, J31 5V, J32 5V, J33 5V, J34 5V, J35 5V, J36 5V, J37 5V, J38 5V, J39 5V, J4 5V, J40 5V, J41 Conn_01x08_MountingPin, J42 Conn_01x04_MountingPin, J5 5V, J6 5V, J7 5V, J8 5V, J9 5V, Q5 AP1606, Q6 AP1606

Commit message: journal
Parts:
- removed J1, J2, J31, J35, J36, J37, J38, J39, J40: 5V, lib:small_pad, symbol Connector_Generic:Conn_01x01
- added J9: 5V, lib:small_pad, symbol Connector_Generic:Conn_01x01
- added R24: 510R, Resistor_SMD:R_0201_0603Metric, symbol Device:R
- renumbered J9 to J31, J41 to J35, J42 to J36, Q6 to Q1, Q5 to Q2, R51 to R25, R23 to R26
Connections:
- net BUZZER- is gone; now on net BZ-: Q2.3 (D)
- net CAM is gone; now on net 5v: J3.1 (Pin_1)
- net ELRS_RX is gone; now on net R2: J36.2 (Pin_2)
- net ELRS_TX is gone; now on net T2: J36.1 (Pin_1)
- net VTX is gone; now on net 10v: J19.1 (Pin_1)
- net 10v: no longer J27.1 (Pin_1)
- net 3v3: now also J16.1 (Pin_1); no longer J5.1 (Pin_1)
- net 5v: now also J17.1 (Pin_1), J24.1 (Pin_1), J26.1 (Pin_1), J4.1 (Pin_1); no longer J20.1 (Pin_1), J23.1 (Pin_1), J7.1 (Pin_1)
- net BAT: now also J15.1 (Pin_1); no longer J26.1 (Pin_1)
- net BZ-: now also J21.1 (Pin_1); no longer J13.1 (Pin_1)
- net CC: now also R24.2; no longer J4.1 (Pin_1)
- net CUR: no longer J34.1 (Pin_1)
- net G: now also J20.1 (Pin_1), J23.1 (Pin_1), J29.1 (Pin_1), J33.1 (Pin_1), J5.1 (Pin_1), J7.1 (Pin_1); no longer J21.1 (Pin_1), J24.1 (Pin_1), J28.1 (Pin_1), J6.1 (Pin_1)
- net LED_STRIP: now also J32.1 (Pin_1)
- net R2: now also J25.1 (Pin_1), J28.1 (Pin_1), J34.1 (Pin_1); no longer J14.1 (Pin_1), J32.1 (Pin_1), J8.1 (Pin_1)
- net R3: now also J13.1 (Pin_1); no longer J11.1 (Pin_1)
- net R6: now also J11.1 (Pin_1); no longer J25.1 (Pin_1)
- net SCL: now also J10.1 (Pin_1); no longer J16.1 (Pin_1)
- net SDA: now also J6.1 (Pin_1); no longer J15.1 (Pin_1)
- net T1: now also J27.1 (Pin_1); no longer J29.1 (Pin_1)
- net T3: now also J9.1 (Pin_1); no longer J10.1 (Pin_1)
- net T6: now also J14.1 (Pin_1); no longer J17.1 (Pin_1)
- net TEL: no longer J33.1 (Pin_1)
- net BZ+: no longer names the net of J12.1 (Pin_1)
- net BZ+: now also R24.1
- net LED renamed VTX_OUT
- net LED_STRIP_L renamed NEOPIXELS
- new net CAM_IN: J8.1 (Pin_1)
Other:
- note added: "Buzzer"
- note added: "bz+"
- moved on the sheet: Q1, Q2, R25, R26
