File: kicad/power.kicad_sch (KiCad schematic)
At the start: 29 parts, among them U2 TLV75733PDBV, U3 LMR51430, U4 LMR51430, U5 TPS2116DRLR

Commit message: journal
Parts:
- added C11: 22uF, Capacitor_SMD:C_0402_1005Metric, symbol Device:C
- added C9: 100n, Capacitor_SMD:C_0201_0603Metric, symbol Device:C
- added D6: LED_1_Green, LED_SMD:LED_0402_1005Metric, symbol Device:LED
- added R10: 510R, Resistor_SMD:R_0201_0603Metric, symbol Device:R
- added U5: TLV75733PDBV, Package_TO_SOT_SMD:SOT-23-5, symbol Regulator_Linear:TLV75733PDBV
- renumbered C24 to C1, C30 to C10, C25 to C2, C32 to C3, C34 to C4, C26 to C5, C27 to C6, C28 to C7, C29 to C8, D7 to D1, D4 to D2, D5 to D3, D3 to D4, D6 to D5, L2 to L1, L3 to L2, R36 to R1, R29 to R2, R30 to R3, R31 to R4, R32 to R5, R27 to R6, R28 to R7, R33 to R8, R34 to R9, U2 to U1, U3 to U2, U4 to U3, U5 to U4
Connections:
- net +5V: now also C9.1, U5.1 (IN), U5.3 (EN)
- net GND: now also C11.2, C9.2, D6.1 (K), U5.2 (GND)
- new net: D6.2 (A), R10.2
- new net +3.3VA: C11.1, R10.1, U5.5 (OUT)
