File: kicad/sensors.kicad_sch (KiCad schematic)
At the start: 8 parts, among them U6 ICM-42688-P, U7 BMP280

Commit message: journal
Parts:
- U6: footprint ICM-42688-P:PQFN50P300X250X97-14N -> ICM_42688_P:PQFN50P300X250X97-14N
- renumbered C36 to C12, C38 to C13, C37 to C14, C39 to C15, R49 to R11, R50 to R12
Changed lines of the file:
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@@
 		(dnp no)
 		(fields_autoplaced yes)
-		(property "Reference" "#PWR0134"
+		(property "Reference" "#PWR036"
 			(at 186.69 105.41 0)
 			(hide yes)
@@
 			(project "Dreamscape-F405-2020"
 				(path "/97210a04-f116-4730-b66b-a4a0966edab8/9a3d92d9-8ad2-49ca-9012-4fac0f59016a"
-					(reference "#PWR0134")
+					(reference "#PWR036")
 					(unit 1)
 				)
@@
 		(dnp no)
 		(fields_autoplaced yes)
-		(property "Reference" "#PWR0131"
+		(property "Reference" "#PWR030"
 			(at 172.72 54.61 0)
 			(hide yes)
@@
 			(project "Dreamscape-F405-2020"
 				(path "/97210a04-f116-4730-b66b-a4a0966edab8/9a3d92d9-8ad2-49ca-9012-4fac0f59016a"
-					(reference "#PWR0131")
+					(reference "#PWR030")
 					(unit 1)
 				)
@@
 			)
 		)
-		(property "Footprint" "ICM-42688-P:PQFN50P300X250X97-14N"
+		(property "Footprint" "ICM_42688_P:PQFN50P300X250X97-14N"
 			(at 132.08 49.53 0)
 			(hide yes)
@@
 		(in_pos_files yes)
 		(dnp no)
-		(property "Reference" "C39"
+		(property "Reference" "C15"
 			(at 186.69 92.71 0)
 			(show_name no)
@@
 			(project "Dreamscape-F405-2020"
 				(path "/97210a04-f116-4730-b66b-a4a0966edab8/9a3d92d9-8ad2-49ca-9012-4fac0f59016a"
-					(reference "C39")
+					(reference "C15")
 					(unit 1)
 				)
@@
 		(dnp no)
 		(fields_autoplaced yes)
-		(property "Reference" "#PWR018"
+		(property "Reference" "#PWR031"
 			(at 175.26 92.71 0)
 			(hide yes)
@@
 			(project "Dreamscape-F405-2020"
 				(path "/97210a04-f116-4730-b66b-a4a0966edab8/9a3d92d9-8ad2-49ca-9012-4fac0f59016a"
-					(reference "#PWR018")
+					(reference "#PWR031")
 					(unit 1)
 				)
@@
 		(dnp no)
 		(fields_autoplaced yes)
-		(property "Reference" "#PWR014"
+		(property "Reference" "#PWR027"
 			(at 158.75 72.39 0)
 			(hide yes)
@@
 			(project "Dreamscape-F405-2020"
 				(path "/97210a04-f116-4730-b66b-a4a0966edab8/9a3d92d9-8ad2-49ca-9012-4fac0f59016a"
-					(reference "#PWR014")
+					(reference "#PWR027")
 					(unit 1)
 				)
@@
 		(dnp no)
 		(fields_autoplaced yes)
-		(property "Reference" "#PWR017"
+		(property "Reference" "#PWR028"
 			(at 158.75 116.84 0)
 			(hide yes)
@@
 			(project "Dreamscape-F405-2020"
 				(path "/97210a04-f116-4730-b66b-a4a0966edab8/9a3d92d9-8ad2-49ca-9012-4fac0f59016a"
-					(reference "#PWR017")
+					(reference "#PWR028")
 					(unit 1)
 				)
@@
 		(dnp no)
 		(fields_autoplaced yes)
-		(property "Reference" "#PWR016"
+		(property "Reference" "#PWR033"
 			(at 184.15 39.37 0)
 			(hide yes)
@@
 			(project "Dreamscape-F405-2020"
 				(path "/97210a04-f116-4730-b66b-a4a0966edab8/9a3d92d9-8ad2-49ca-9012-4fac0f59016a"
-					(reference "#PWR016")
+					(reference "#PWR033")
 					(unit 1)
 				)
@@
 		(dnp no)
 		(fields_autoplaced yes)
-		(property "Reference" "#PWR0132"
+		(property "Reference" "#PWR034"
 			(at 184.15 54.61 0)
 			(hide yes)
@@
 			(project "Dreamscape-F405-2020"
 				(path "/97210a04-f116-4730-b66b-a4a0966edab8/9a3d92d9-8ad2-49ca-9012-4fac0f59016a"
-					(reference "#PWR0132")
+					(reference "#PWR034")
 					(unit 1)
 				)
@@
 		(dnp no)
 		(fields_autoplaced yes)
-		(property "Reference" "#PWR0133"
+		(property "Reference" "#PWR032"
 			(at 175.26 105.41 0)
 			(hide yes)
@@
 			(project "Dreamscape-F405-2020"
 				(path "/97210a04-f116-4730-b66b-a4a0966edab8/9a3d92d9-8ad2-49ca-9012-4fac0f59016a"
-					(reference "#PWR0133")
+					(reference "#PWR032")
 					(unit 1)
 				)
@@
 		(in_pos_files yes)
 		(dnp no)
-		(property "Reference" "C37"
+		(property "Reference" "C14"
 			(at 184.15 41.91 0)
 			(show_name no)
@@
 			(project "Dreamscape-F405-2020"
 				(path "/97210a04-f116-4730-b66b-a4a0966edab8/9a3d92d9-8ad2-49ca-9012-4fac0f59016a"
-					(reference "C37")
+					(reference "C14")
 					(unit 1)
 				)
@@
 		(in_pos_files yes)
 		(dnp no)
-		(property "Reference" "R50"
+		(property "Reference" "R12"
 			(at 130.048 106.426 90)
 			(show_name no)
@@
 			(project "Dreamscape-F405-2020"
 				(path "/97210a04-f116-4730-b66b-a4a0966edab8/9a3d92d9-8ad2-49ca-9012-4fac0f59016a"
-					(reference "R50")
+					(reference "R12")
 					(unit 1)
 				)
@@
 		(dnp no)
 		(fields_autoplaced yes)
-		(property "Reference" "#PWR019"
+		(property "Reference" "#PWR035"
 			(at 186.69 90.17 0)
 			(hide yes)
@@
 			(project "Dreamscape-F405-2020"
 				(path "/97210a04-f116-4730-b66b-a4a0966edab8/9a3d92d9-8ad2-49ca-9012-4fac0f59016a"
-					(reference "#PWR019")
+					(reference "#PWR035")
 					(unit 1)
 				)
@@
 		(in_pos_files yes)
 		(dnp no)
-		(property "Reference" "C36"
+		(property "Reference" "C12"
 			(at 172.72 41.91 0)
 			(show_name no)
@@
 			(project "Dreamscape-F405-2020"
 				(path "/97210a04-f116-4730-b66b-a4a0966edab8/9a3d92d9-8ad2-49ca-9012-4fac0f59016a"
-					(reference "C36")
+					(reference "C12")
 					(unit 1)
 				)
@@
 		(in_pos_files yes)
 		(dnp no)
-		(property "Reference" "C38"
+		(property "Reference" "C13"
 			(at 175.26 92.71 0)
 			(show_name no)
@@
 			(project "Dreamscape-F405-2020"
 				(path "/97210a04-f116-4730-b66b-a4a0966edab8/9a3d92d9-8ad2-49ca-9012-4fac0f59016a"
-					(reference "C38")
+					(reference "C13")
 					(unit 1)
 				)
@@
 		(in_pos_files yes)
 		(dnp no)
-		(property "Reference" "R49"
+		(property "Reference" "R11"
 			(at 89.408 45.974 90)
 			(show_name no)
@@
 			(project "Dreamscape-F405-2020"
 				(path "/97210a04-f116-4730-b66b-a4a0966edab8/9a3d92d9-8ad2-49ca-9012-4fac0f59016a"
-					(reference "R49")
+					(reference "R11")
 					(unit 1)
 				)
@@
 		(dnp no)
 		(fields_autoplaced yes)
-		(property "Reference" "#PWR0156"
+		(property "Reference" "#PWR025"
 			(at 87.63 43.18 0)
 			(hide yes)
@@
 			(project "Dreamscape-F405-2020"
 				(path "/97210a04-f116-4730-b66b-a4a0966edab8/9a3d92d9-8ad2-49ca-9012-4fac0f59016a"
-					(reference "#PWR0156")
+					(reference "#PWR025")
 					(unit 1)
 				)
@@
 		(dnp no)
 		(fields_autoplaced yes)
-		(property "Reference" "#PWR015"
+		(property "Reference" "#PWR029"
 			(at 172.72 41.91 0)
 			(hide yes)
@@
 			(project "Dreamscape-F405-2020"
 				(path "/97210a04-f116-4730-b66b-a4a0966edab8/9a3d92d9-8ad2-49ca-9012-4fac0f59016a"
-					(reference "#PWR015")
+					(reference "#PWR029")
 					(unit 1)
 				)
@@
 		(dnp no)
 		(fields_autoplaced yes)
-		(property "Reference" "#PWR0157"
+		(property "Reference" "#PWR026"
 			(at 128.27 109.22 0)
 			(hide yes)
@@
 			(project "Dreamscape-F405-2020"
 				(path "/97210a04-f116-4730-b66b-a4a0966edab8/9a3d92d9-8ad2-49ca-9012-4fac0f59016a"
-					(reference "#PWR0157")
-					(unit 1)
-				)
+					(reference "#PWR026")
+					(unit 1)
+				)
