File: kicad/stm32.kicad_sch (KiCad schematic)
At the start: 11 parts, among them U1 STM32F405VGTx

Commit message: journal
Parts:
- added C17, C19, C21, C26, C27: 100n, Capacitor_SMD:C_0201_0603Metric, symbol Device:C
- added C22, C24: 20pF, Capacitor_SMD:C_0201_0603Metric, symbol Device:C
- added J1, J2: 5V, lib:small_pad, symbol Connector_Generic:Conn_01x01
- added R14, R15: 5.1k, Resistor_SMD:R_0201_0603Metric, symbol Device:R
- added R16, R17: 10k, Resistor_SMD:R_0201_0603Metric, symbol Device:R
- added R21: 1k, Resistor_SMD:R_0201_0603Metric, symbol Device:R
- added U11, U12: TS2306A 240GF MSM 9_C2976675, lib:SW-SMD_4P-L3.0-W2.0-P0.85-LS3.5, symbol lib:TS2306A240GFMSM9_C2976675
- added X1: X32258MOB4SI, lib:CRYSTAL-SMD_4P-L2.5-W2.0-BL-A, symbol lib:XTM25012000JT00351001
- renumbered C2 to C18, C1 to C20, C4 to C23, C22 to C25, D2 to D7, R1 to R18, R2 to R19, R9 to R20, R52 to R22, R53 to R23, U1 to U9
Connections:
- net SPI1_MISO is gone; now on net SPI1.MISO: U9.31 (PA6)
- net SPI1_MOSI is gone; now on net SPI1.MOSI: U9.32 (PA7)
- net SPI1_SCK is gone; now on net SPI1.SCK: U9.30 (PA5)
- net SPI2_MISO is gone; now on net SPI2.MISO: U9.53 (PB14)
- net SPI2_MOSI is gone; now on net SPI2.MOSI: U9.54 (PB15)
- net SPI2_SCK is gone; now on net SPI2.SCK: U9.52 (PB13)
- net SPI3_MISO is gone; now on net SPI3.MISO: U9.79 (PC11)
- net SPI3_MOSI is gone; now on net SPI3.MOSI: U9.80 (PC12)
- net SPI3_SCK is gone; now on net SPI3.SCK: U9.78 (PC10)
- net ADC_VBAT: now also U9.15 (PC0)
- net ESC_CURR: now also U9.16 (PC1)
- net GND: now also C17.1, C19.1, C21.1, C22.1, C24.1, C26.1, C27.1, R17.2, U11.1, X1.2 (GND), X1.4 (GND)
- net LED0: now also U9.95 (PB8)
- net +3.3V: now reaches U9.100 (VDD)
- net +3.3V: now also U9.11 (VDD), U9.19 (VDD), U9.28 (VDD), U9.50 (VDD), U9.6 (VBAT), U9.75 (VDD), C19.2, C26.2, C27.2, R14.1, R15.1, R16.1, U12.2
- net XIN: now reaches U9.12 (PH0)
- net XIN: now also C22.2, X1.1
- net XOUT: now reaches U9.13 (PH1)
- net XOUT: now also R21.1
- net NRST: now reaches U9.14 (NRST)
- net NRST: now also R16.2, U11.2
- net +3.3VA: now reaches U9.21 (VREF+)
- net +3.3VA: now also U9.22 (VDDA), C17.2, C21.2
- net CC: now reaches U9.23 (PA0)
- net TEL: now reaches U9.24 (PA1)
- net T2: now reaches U9.25 (PA2)
- net R2: now reaches U9.26 (PA3)
- net T3: now reaches U9.47 (PB10)
- net R3: now reaches U9.48 (PB11)
- net M1: now reaches U9.59 (PD12)
- net M2: now reaches U9.60 (PD13)
- net M3: now reaches U9.61 (PD14)
- net M4: now reaches U9.62 (PD15)
- net T6: now reaches U9.63 (PC6)
- net R6: now reaches U9.64 (PC7)
- net SDA: now reaches U9.65 (PC8)
- net SDA: now also R14.2
- net SCL: now reaches U9.66 (PC9)
- net SCL: now also R15.2
- net D-: now reaches U9.70 (PA11)
- net D+: now reaches U9.71 (PA12)
- net SWDIO: now reaches U9.72 (PA13)
- net SWDIO: now also J2.1 (Pin_1)
- net SWCLK: now reaches U9.76 (PA14)
- net SWCLK: now also J1.1 (Pin_1)
- net LED_STRIP: now reaches U9.89 (PB3)
- net BEEPER: now reaches U9.91 (PB5)
- net T1: now reaches U9.92 (PB6)
- net R1: now reaches U9.93 (PB7)
- net BOOT0: now reaches U9.94 (BOOT0)
- net BOOT0: now also R17.1, U12.1
- new net: C24.2, R21.2, X1.3
Other:
- moved on the sheet: C18, C20, C25, R20, U9

Commit message: small changes
Connections:
- net SCL: now also R14.2, U9.67 (PA8); no longer R15.2, U9.66 (PC9)
- net SDA: now also R15.2, U9.66 (PC9); no longer R14.2, U9.65 (PC8)
Other:
- moved on the sheet: R14
Changed lines of the file:
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@@
 	)
 	(junction
-		(at 137.16 157.48)
-		(diameter 0)
-		(color 0 0 0 0)
-	)
-	(junction
 		(at 39.37 60.96)
 		(diameter 0)
@@
 	)
 	(junction
+		(at 129.54 71.12)
+		(diameter 0)
+		(color 0 0 0 0)
+	)
+	(junction
 		(at 260.35 53.34)
 		(diameter 0)
@@
 	(wire
 		(pts
-			(xy 137.16 157.48) (xy 137.16 151.13)
+			(xy 129.54 71.12) (xy 129.54 64.77)
 		)
 		(stroke
@@
 	(wire
 		(pts
-			(xy 153.67 151.13) (xy 160.02 151.13)
+			(xy 146.05 64.77) (xy 152.4 64.77)
 		)
 		(stroke
@@
 	(wire
 		(pts
-			(xy 137.16 151.13) (xy 146.05 151.13)
+			(xy 129.54 64.77) (xy 138.43 64.77)
 		)
 		(stroke
@@
 		)
 	)
+	(wire
+		(pts
+			(xy 114.3 71.12) (xy 129.54 71.12)
+		)
+		(stroke
+			(width 0)
+			(type default)
+		)
+	)
 	(bus
 		(pts
@@
 	(wire
 		(pts
-			(xy 148.59 157.48) (xy 137.16 157.48)
+			(xy 140.97 71.12) (xy 129.54 71.12)
 		)
 		(stroke
@@
 	(wire
 		(pts
-			(xy 114.3 157.48) (xy 137.16 157.48)
-		)
-		(stroke
-			(width 0)
-			(type default)
-		)
-	)
-	(wire
-		(pts
 			(xy 115.57 154.94) (xy 114.3 154.94)
 		)
@@
 		)
 	)
-	(hierarchical_label "SCL"
+	(hierarchical_label "SDA"
 		(shape input)
 		(at 148.59 160.02 0)
@@
 		)
 	)
-	(hierarchical_label "SDA"
+	(hierarchical_label "SCL"
 		(shape input)
-		(at 148.59 157.48 0)
+		(at 140.97 71.12 0)
 		(effects
 			(font
@@
 	(symbol
 		(lib_id "power:+3.3V")
-		(at 160.02 151.13 270)
+		(at 152.4 64.77 270)
 		(unit 1)
 		(body_style 1)
@@
 		(fields_autoplaced yes)
 		(property "Reference" "#PWR056"
-			(at 156.21 151.13 0)
+			(at 148.59 64.77 0)
 			(hide yes)
 			(show_name no)
@@
 		)
 		(property "Value" "+3.3V"
-			(at 163.83 151.1299 90)
+			(at 156.21 64.7699 90)
 			(show_name no)
 			(do_not_autoplace no)
@@
 		)
 		(property "Footprint" ""
-			(at 160.02 151.13 0)
+			(at 152.4 64.77 0)
 			(hide yes)
 			(show_name no)
@@
 		)
 		(property "Datasheet" ""
-			(at 160.02 151.13 0)
+			(at 152.4 64.77 0)
 			(hide yes)
 			(show_name no)
@@
 		)
 		(property "Description" "Power symbol creates a global label with name \"+3.3V\""
-			(at 160.02 151.13 0)
+			(at 152.4 64.77 0)
 			(hide yes)
 			(show_name no)
@@
 	(symbol
 		(lib_id "Device:R")
-		(at 149.86 151.13 270)
+		(at 142.24 64.77 270)
 		(unit 1)
 		(body_style 1)
@@
 		(dnp no)
 		(property "Reference" "R14"
-			(at 147.574 148.082 90)
+			(at 139.954 61.722 90)
 			(show_name no)
 			(do_not_autoplace no)
@@
 		)
 		(property "Value" "5.1k"
-			(at 152.146 148.082 90)
+			(at 144.526 61.722 90)
 			(show_name no)
 			(do_not_autoplace no)
@@
 		)
 		(property "Footprint" "Resistor_SMD:R_0201_0603Metric"
-			(at 149.86 149.352 90)
+			(at 142.24 62.992 90)
 			(hide yes)
 			(show_name no)
@@
 		)
 		(property "Datasheet" ""
-			(at 149.86 151.13 0)
+			(at 142.24 64.77 0)
 			(hide yes)
 			(show_name no)
@@
 		)
 		(property "Description" "Resistor"
-			(at 149.86 151.13 0)
+			(at 142.24 64.77 0)
 			(hide yes)
 			(show_name no)
@@
 		)
 		(property "LCSC" "C270344"
-			(at 149.86 151.13 90)
+			(at 142.24 64.77 90)
 			(hide yes)
 			(show_name no)
@@
 		)
 		(property "MPN" "0201WMF5101TEE"
-			(at 71.12 -57.15 0)
+			(at 63.5 -143.51 0)
 			(hide yes)
 			(show_name no)
@@
 		)
 		(property "Manufacturer" "UNI-ROYAL"
-			(at 71.12 -57.15 0)
+			(at 63.5 -143.51 0)
 			(hide yes)
 			(show_name no)
